File: hardware/ATMEGA16M1.sch (KiCad schematic (older format))
At the start: 56 parts, among them J1 PWR, J2 USB, J3 RELAY1, J4 RELAY2, J5 RELAY3, J6 GPIO, J7 AMP/D2A, J8 ADC, J9 CAN, SW1 RESET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

Commit message: Updated schematic for JGB
Parts:
- removed JP1: JUMPER3, ~, symbol JUMPER3
- C1, C2, C3, C4, C5, C6, C7, C8: symbol C -> C-RESCUE-ATMEGA16M1
- D1: symbol LED -> LED-RESCUE-ATMEGA16M1; P/N 732-4982-1-ND -> 475-1410-1-ND; URL http://www.digikey.com/product-detail/en/150080BS75000/732-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 -> http://www.digikey.com/product-detail/en/osram-opto-semicon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
- D2, D3, D4, D5, D6, D7, D8: symbol LED -> LED-RESCUE-ATMEGA16M1
- R1, R10, R11, R12, R13, R14, R15, R16, R2, R3, R4, R5, R6, R7, R8, R9: symbol R -> R-RESCUE-ATMEGA16M1
- U4: symbol MCP2551-I/SN -> MCP2551-I/SN-RESCUE-ATMEGA16M1
Connections:
- net V_USER is gone; now on net V_GLV: C2.1, U1.3 (VI)
Other:
- note added: "Removed USB connection\nWe need 24V now"
Changed lines of the file:
@@
 EESchema Schematic File Version 2
+LIBS:ATMEGA16M1-rescue
 LIBS:power
 LIBS:device
@@
 LIBS:memory
 LIBS:xilinx
-LIBS:special
 LIBS:microcontrollers
 LIBS:dsp
@@
 LIBS:contrib
 LIBS:valves
-LIBS:w_connectors
-LIBS:w_relay
-LIBS:w_vacuum
-LIBS:w_transistor
-LIBS:w_rtx
-LIBS:w_opto
-LIBS:w_microcontrollers
-LIBS:w_memory
-LIBS:w_logic
-LIBS:w_device
-LIBS:w_analog
 LIBS:custom
 LIBS:dips-s
 LIBS:ATMEGA16M1-cache
-EELAYER 27 0
+EELAYER 25 0
 EELAYER END
 $Descr USLetter 11000 8500
@@
 $EndComp
 $Comp
-L GND #PWR02
+L GND-RESCUE-ATMEGA16M1 #PWR02
 U 1 1 54DAA08D
 P 3650 4250
@@
 $EndComp
 $Comp
-L C C7
+L C-RESCUE-ATMEGA16M1 C7
 U 1 1 54DAA126
 P 6100 4750
@@
 $EndComp
 $Comp
-L C C8
+L C-RESCUE-ATMEGA16M1 C8
 U 1 1 54DAA13D
 P 6700 4750
@@
 $EndComp
 $Comp
-L GND #PWR03
+L GND-RESCUE-ATMEGA16M1 #PWR03
 U 1 1 54DAA197
 P 6400 5250
@@
 GND
 $Comp
-L R R4
+L R-RESCUE-ATMEGA16M1 R4
 U 1 1 54DAA28F
 P 5100 5700
@@
 $EndComp
 $Comp
-L GND #PWR05
+L GND-RESCUE-ATMEGA16M1 #PWR05
 U 1 1 54DAA320
 P 5550 6100
@@
 $EndComp
 $Comp
-L C C2
+L C-RESCUE-ATMEGA16M1 C2
 U 1 1 54DAA5A1
 P 1300 1650
@@
 $EndComp
 $Comp
-L C C3
+L C-RESCUE-ATMEGA16M1 C3
 U 1 1 54DAA662
 P 2350 1650
@@
 $EndComp
 $Comp
-L GND #PWR06
+L GND-RESCUE-ATMEGA16M1 #PWR06
 U 1 1 54DAA728
 P 1850 2050
@@
 V_USER
 $Comp
-L LED D1
+L LED-RESCUE-ATMEGA16M1 D1
 U 1 1 54DAF1B3
 P 1700 2800
@@
 F 2 "~" H 1700 2800 60  0000 C CNN
 F 3 "~" H 1700 2800 60  0000 C CNN
-F 4 "732-4982-1-ND" H 1700 2800 60  0001 C CNN "P/N"
+F 4 "475-1410-1-ND" H 1700 2800 60  0001 C CNN "P/N"
 F 5 "Digikey" H 1700 2800 60  0001 C CNN "Supplier"
-F 6 "http://www.digikey.com/product-detail/en/150080BS75000/732-4982-1-ND/4489910" H 1700 2800 60  0001 C CNN "URL"
+F 6 "http://www.digikey.com/product-detail/en/osram-opto-semiconductors-inc/LG-R971-KN-1/475-1410-1-ND/1802598" H 1700 2800 60  0001 C CNN "URL"
 	1    1700 2800
 	1    0    0    -1
 $EndComp
 $Comp
-L R R1
+L R-RESCUE-ATMEGA16M1 R1
 U 1 1 54DAF85C
 P 1150 2800
@@
 $EndComp
 $Comp
-L GND #PWR09
+L GND-RESCUE-ATMEGA16M1 #PWR09
 U 1 1 54DAF9E0
 P 2000 2900
@@
 $EndComp
 $Comp
-L C C5
+L C-RESCUE-ATMEGA16M1 C5
 U 1 1 54DBBDE0
 P 3300 1900
@@
 $EndComp
 $Comp
-L GND #PWR010
+L GND-RESCUE-ATMEGA16M1 #PWR010
 U 1 1 54DBBF13
 P 3300 2200
@@
 FTDI_RX
 $Comp
-L C C4
+L C-RESCUE-ATMEGA16M1 C4
 U 1 1 54DE19D6
 P 2600 1650
@@
 ATMEGA 16M1 MICROCONTROLLER
 $Comp
-L MCP2551-I/SN U4
+L MCP2551-I/SN-RESCUE-ATMEGA16M1 U4
 U 1 1 54EE8E2B
 P 8150 5700
@@
 CANRX
 $Comp
-L R R12
+L R-RESCUE-ATMEGA16M1 R12
 U 1 1 54EE9FDE
 P 7500 6250
@@
 $EndComp
 $Comp
-L GND #PWR011
+L GND-RESCUE-ATMEGA16M1 #PWR011
 U 1 1 54EEA1CE
 P 7500 6600
@@
 FTDI_TX
 $Comp
-L R R14
+L R-RESCUE-ATMEGA16M1 R14
 U 1 1 54EEA853
 P 8050 3750
@@
 $EndComp
 $Comp
-L R R6
+L R-RESCUE-ATMEGA16M1 R6
 U 1 1 54EEA92A
 P 5250 7000
@@
 $EndComp
 $Comp
-L LED D3
+L LED-RESCUE-ATMEGA16M1 D3
 U 1 1 54EEA931
 P 4700 7000
@@
 $EndComp
 $Comp
-L GND #PWR012
+L GND-RESCUE-ATMEGA16M1 #PWR012
 U 1 1 54EEAF05
 P 2000 6600
@@
 $EndComp
 $Comp
-L C C1
+L C-RESCUE-ATMEGA16M1 C1
 U 1 1 54EEB93E
 P 850 5500
@@
 $EndComp
 $Comp
-L GND #PWR015
+L GND-RESCUE-ATMEGA16M1 #PWR015
 U 1 1 54EEB94D
 P 850 5800
@@
 $EndComp
 $Comp
-L R R7
+L R-RESCUE-ATMEGA16M1 R7
 U 1 1 54EEBC81
 P 4750 7300
@@
 $EndComp
 $Comp
-L LED D4
+L LED-RESCUE-ATMEGA16M1 D4
 U 1 1 54EEBC88
 P 5300 7300
@@
 CANTX
 $Comp
-L R R8
+L R-RESCUE-ATMEGA16M1 R8
 U 1 1 54EEBC91
 P 4750 7600
@@
 $EndComp
 $Comp
-L LED D5
+L LED-RESCUE-ATMEGA16M1 D5
 U 1 1 54EEBC98
 P 5300 7600
@@
 AC/DC Relay
 $Comp
-L GND #PWR016
+L GND-RESCUE-ATMEGA16M1 #PWR016
 U 1 1 54F3FAF1
 P 7450 1500
@@
 $EndComp
 $Comp
-L GND #PWR017
+L GND-RESCUE-ATMEGA16M1 #PWR017
 U 1 1 54F3FBDE
 P 7450 2200
@@
 NoConn ~ 8800 1950
 $Comp
-L C C6
+L C-RESCUE-ATMEGA16M1 C6
 U 1 1 54F5ED52
 P 3650 2250
@@
 $EndComp
 $Comp
-L GND #PWR018
+L GND-RESCUE-ATMEGA16M1 #PWR018
 U 1 1 54F5EF3F
 P 3650 2550
@@
 $EndComp
 $Comp
-L GND #PWR020
+L GND-RESCUE-ATMEGA16M1 #PWR020
 U 1 1 54FEFEDB
 P 8150 6200
@@
 	1    0    0    -1
 $EndComp
-$Comp
-L JUMPER3 JP1
-U 1 1 54FF01E2
-P 2250 900
-F 0 "JP1" H 2300 800 40  0000 L CNN
-F 1 "JUMPER3" H 2250 1000 40  0000 C CNN
-F 2 "~" H 2250 900 60  0000 C CNN
-F 3 "~" H 2250 900 60  0000 C CNN
-F 4 "952-2264-ND" H 2250 900 60  0001 C CNN "P/N"
-F 5 "Digikey" H 2250 900 60  0001 C CNN "Supplier"
-F 6 "http://www.digikey.com/product-detail/en/M20-9990346/952-2264-ND/3728228" H 2250 900 60  0001 C CNN "URL"
-	1    2250 900
-	1    0    0    -1
-$EndComp
 Text Label 1600 900  0    60   ~ 0
 V_GLV
-Text Label 2900 900  2    60   ~ 0
-V_USB
 Text Label 1600 1100 0    60   ~ 0
 V_USER
@@
 POWER LED
 $Comp
-L R R9
+L R-RESCUE-ATMEGA16M1 R9
 U 1 1 55161CE8
 P 7200 1100
@@
 $EndComp
 $Comp
-L R R10
+L R-RESCUE-ATMEGA16M1 R10
 U 1 1 55161DD0
 P 7200 1800
@@
 GND
 $Comp
-L R R11
+L R-RESCUE-ATMEGA16M1 R11
 U 1 1 55161DCA
 P 7200 2500
@@
 SSR2
 $Comp
-L GND #PWR024
+L GND-RESCUE-ATMEGA16M1 #PWR024
 U 1 1 54F5ECFA
 P 7450 2900
@@
 $EndComp
 $Comp
-L R R13
+L R-RESCUE-ATMEGA16M1 R13
 U 1 1 551C5383
 P 8050 3450
@@
 $EndComp
 $Comp
-L LED D6
+L LED-RESCUE-ATMEGA16M1 D6
 U 1 1 551C5389
 P 8950 3450
@@
 SSR0
 $Comp
-L R R15
+L R-RESCUE-ATMEGA16M1 R15
 U 1 1 551C5393
 P 8050 4050
@@
 	4100 5300 5700 5300
 Wire Wire Line
-	2000 900  1600 900
-Wire Wire Line
-	2500 900  2900 900
-Wire Wire Line
-	2250 1000 2250 1100
+	1600 900  2250 900
+Wire Wire Line
+	2250 900  2250 1100
 Wire Wire Line
 	2250 1100 1600 1100
@@
 Connection ~ 9350 4050
 $Comp
-L GND #PWR025
+L GND-RESCUE-ATMEGA16M1 #PWR025
 U 1 1 551C5842
 P 9350 4150
@@
 $EndComp
 $Comp
-L LED D7
+L LED-RESCUE-ATMEGA16M1 D7
 U 1 1 551C5892
 P 8950 3750
@@
 $EndComp
 $Comp
-L LED D8
+L LED-RESCUE-ATMEGA16M1 D8
 U 1 1 551C5898
 P 8950 4050
@@
 $EndComp
 $Comp
-L R R5
+L R-RESCUE-ATMEGA16M1 R5
 U 1 1 551C5A61
 P 5250 6700
@@
 $EndComp
 $Comp
-L LED D2
+L LED-RESCUE-ATMEGA16M1 D2
 U 1 1 551C5A67
 P 4700 6700
@@
 JP1 Jumper Shunt\nP/N: S9001-ND\nSupplier: Digikey
 $Comp
-L R R16
+L R-RESCUE-ATMEGA16M1 R16
 U 1 1 55284A3E
 P 9200 5700
@@
 	1100 7600 1900 7600
 $Comp
-L R R2
+L R-RESCUE-ATMEGA16M1 R2
 U 1 1 55289115
 P 2150 7400
@@
 $EndComp
 $Comp
-L R R3
+L R-RESCUE-ATMEGA16M1 R3
 U 1 1 5528913C
 P 2150 7600
@@
 Connection ~ 5700 7600
 $Comp
-L GND #PWR026
+L GND-RESCUE-ATMEGA16M1 #PWR026
 U 1 1 5528A485
 P 5700 7700
@@
 	1    0    0    -1
 $EndComp
+Text Notes 1800 750  0    60   ~ 0
+Removed USB connection\nWe need 24V now
 $EndSCHEMATC
